Commit message: Update mini_pupper.urdf

File: 01 - IK/mini_pupper.urdf (robot description, URDF)
Before this commit: robot mini_pupper, 13 links, 12 joints
Links:
- added link FL-foot
- added link FR-foot
- added link RL-foot
- added link RR-foot
Joints:
- added joint FL-FOOT: type fixed, parent FL-tibia, child FL-foot, origin xyz=0.060 0 0 rpy=0 0 0, axis 0 0 1
- added joint FR-FOOT: type fixed, parent FR-tibia, child FR-foot, origin xyz=0.060 0 0 rpy=0 0 0, axis 0 0 1
- added joint RL-FOOT: type fixed, parent RL-tibia, child RL-foot, origin xyz=0.060 0 0 rpy=0 0 0, axis 0 0 1
- added joint RR-FOOT: type fixed, parent RR-tibia, child RR-foot, origin xyz=0.060 0 0 rpy=0 0 0, axis 0 0 1

Commit message: fix meshes issue with jupiter lab

File: 01 - IK/mini_pupper.urdf (robot description, URDF)
Before this commit: robot mini_pupper, 17 links, 16 joints
Links:
- link FL-femur: geometry collision box size=0.054 0.007 0.002; visual box size=0.056 0.007 0.002
- link FL-pod: geometry collision box size=0.031 0.030 0.038; visual box size=0.031 0.030 0.038
- link FL-tibia: geometry collision box size=0.060 0.006 0.002; visual box size=0.060 0.006 0.002
- link FR-femur: geometry collision box size=0.056 0.007 0.002; visual box size=0.056 0.007 0.002
- link FR-pod: geometry collision box size=0.031 0.030 0.038; visual box size=0.031 0.030 0.038
- link FR-tibia: geometry collision box size=0.060 0.006 0.002; visual box size=0.060 0.006 0.002
- link RL-femur: geometry collision box size=0.054 0.007 0.002; visual box size=0.056 0.007 0.002
- link RL-pod: geometry collision box size=0.031 0.030 0.038; visual box size=0.031 0.030 0.038
- link RL-tibia: geometry collision box size=0.060 0.006 0.002; visual box size=0.060 0.006 0.002
- link RR-femur: geometry collision box size=0.054 0.007 0.002; visual box size=0.056 0.007 0.002
- link RR-pod: geometry collision box size=0.031 0.030 0.038; visual box size=0.031 0.030 0.038
- link RR-tibia: geometry collision box size=0.060 0.006 0.002; visual box size=0.060 0.006 0.002
- link base_link: geometry collision box size=0.150 0.036 0.008; collision box size=0.180 0.060 0.045
Joints:
- joint FL-HIPS: origin xyz=0.0 0.019 0.0 rpy=-1.57079 1.57079 0 -> xyz=0.0 0.020 0.0 rpy=-1.57079 1.57079 0
- joint FL-KNEE: origin xyz=0.050 0 0.005 rpy=0 0 0 -> xyz=0.050 0 0.006 rpy=0 0 0
- joint FR-HIPS: origin xyz=0.0 -0.019 0.0 rpy=-1.57079 1.57079 0 -> xyz=0.0 -0.020 0.0 rpy=-1.57079 1.57079 0
- joint FR-KNEE: origin xyz=0.050 0 -0.005 rpy=0 0 0 -> xyz=0.050 0 -0.006 rpy=0 0 0
- joint RL-HIPS: origin xyz=0.0 0.019 0.0 rpy=-1.57079 1.57079 0 -> xyz=0.0 0.020 0.0 rpy=-1.57079 1.57079 0
- joint RL-KNEE: origin xyz=0.050 0 0.005 rpy=0 0 0 -> xyz=0.050 0 0.006 rpy=0 0 0
- joint RR-HIPS: origin xyz=0.0 -0.019 0.0 rpy=-1.57079 1.57079 0 -> xyz=0.0 -0.020 0.0 rpy=-1.57079 1.57079 0
- joint RR-KNEE: origin xyz=0.050 0 -0.005 rpy=0 0 0 -> xyz=0.050 0 -0.006 rpy=0 0 0

Commit message: poses

File: 01 - IK/mini_pupper.urdf (robot description, URDF)
Before this commit: robot mini_pupper, 17 links, 16 joints
Links:
- link base_link: mass 0.2 -> None; geometry collision box size=0.180 0.060 0.045
